Commit message: IsaacSim support (#13)
Fix enactic/openarm_isaac_lab#2

* Change dae file
* Change physical parameter

Reported by @Bakel-Bakel. Thanks!!!

File: urdf/arm/openarm_arm.xacro (robot description, xacro)
@@ -82,10 +82,10 @@
       <xacro:openarm-limits name="joint7" config="${joint_limits}" />
     </joint>
-    <link name="${prefix}link8"/>
+    <!-- <link name="${prefix}link8"/>
     <joint name="${prefix}joint8" type="fixed">
       <xacro:openarm-kinematics name="joint8" config="${kinematics}" />
       <parent link="${prefix}link7" />
       <child link="${prefix}link8" />
-    </joint>
+    </joint> -->
   </xacro:macro>
 </robot>

File: urdf/ee/openarm_hand.xacro (robot description, xacro)
@@ -58,5 +58,5 @@
       <parent link="${ee_prefix}hand" />
       <child link="${ee_prefix}right_finger" />
-      <origin xyz="0 0.00 0.015" rpy="0 0 0" />
+      <origin xyz="0 -0.006 0.015" rpy="0 0 0" />
       <axis xyz="0 -1 0" />
       <limit effort="333" lower="0.0" upper="0.044" velocity="10.0" />
@@ -65,5 +65,5 @@
       <parent link="${ee_prefix}hand" />
       <child link="${ee_prefix}left_finger" />
-      <origin xyz="0 0.012 0.015" rpy="0 0 0" />
+      <origin xyz="0 0.006 0.015" rpy="0 0 0" />
       <axis xyz="0 1 0" />
       <limit effort="333" lower="0.0" upper="0.044" velocity="10.0" />

File: urdf/ee/openarm_hand_arguments.xacro (robot description, xacro)
@@ -4,5 +4,5 @@
   <xacro:arg name="special_connection" default="" />
   <!-- Position offset between ee and parent frame -->
-  <xacro:arg name="xyz_ee" default="0 -0.025 0.1001" />
+  <xacro:arg name="xyz_ee" default="0 -0.0 0.1001" />
   <!-- Rotation offset between ee and parent frame -->
   <xacro:arg name="rpy_ee" default= "0 0 0" />

File: urdf/robot/openarm_robot.xacro (robot description, xacro)
@@ -105,5 +105,5 @@
         <xacro:if value="$(eval hand and ee_type == 'openarm_hand')">
             <xacro:openarm_hand
-                connected_to="openarm_left_link8"
+                connected_to="openarm_left_link7"
                 arm_type="${arm_type}"
                 arm_prefix="left_"
@@ -118,5 +118,5 @@
             />
             <xacro:openarm_hand
-                connected_to="openarm_right_link8"
+                connected_to="openarm_right_link7"
                 arm_type="${arm_type}"
                 arm_prefix="right_"
@@ -157,6 +157,6 @@
         <xacro:if value="${hand and ee_type == 'openarm_hand'}">
         <xacro:property name="special_connection" value="$(arg special_connection)" />
-        <!-- <xacro:property name="connection" value="${special_connection if special_connection != '' else arm_type + '_link8'}" /> -->
-        <xacro:property name="connection" value="${special_connection if special_connection != '' else 'openarm' + '_link8'}" />
+        <!-- <xacro:property name="connection" value="${special_connection if special_connection != '' else arm_type + '_link7'}" /> -->
+        <xacro:property name="connection" value="${special_connection if special_connection != '' else 'openarm' + '_link7'}" />
         <xacro:if value="$(eval hand and ee_type == 'openarm_hand')">
         <xacro:openarm_hand
